Commit message: Added gazebo control. differential drive for now.

File: src/my_bot/description/robot.urdf.xacro (robot description, xacro)
@@ -1,3 +1,5 @@
 <?xml version="1.0"?>
-<robot xmlns:xacro="http://www.ros.org/wiki/xacro"  name="robot">
+<robot xmlns:xacro="http://www.ros.org/wiki/xacro"  name="Assem1">
+  <xacro:include filename="robot_core.xacro"/>
+  <xacro:include filename="gazebo_control.xacro"/>
 </robot>

File: src/my_bot/description/robot_core.xacro (robot description, xacro)
@@ -1,28 +1,28 @@
 <?xml version="1.0" encoding="utf-8"?>
-<robot xmlns:xacro="http://www.ros.org/wiki/xacro" name="Assem1">
+<robot xmlns:xacro="http://www.ros.org/wiki/xacro">
   <!-- ===================== -->
   <!--   LINKS               -->
   <!-- ===================== -->
-<!-- <link name="base_link"></link> -->
+  <link name="base_link"></link>
   <link name="Waist">
     <inertial>
-      <origin xyz="-1.18888240640652E-16 -0.00507058467782265 -0.0187972227348701" rpy="0 0 0"/>
-      <mass value="14.4540071153471"/>
+      <origin xyz="-1.18888240640652E-16 -0.00507058467782265 -0.0187972227348701" rpy="0 0 0" />
+      <mass value="14.4540071153471" />
       <inertia ixx="0.0700688932175611" ixy="-3.86937762023137E-19" ixz="-1.76854570708965E-20"
-               iyy="0.292430846914939" iyz="-1.32037216353675E-18" izz="0.292430846914939"/>
-    </inertial>
-    <visual>
-      <origin xyz="0 0 0" rpy="0 0 0"/>
-      <geometry>
-        <mesh filename="file://$(find bpwr)/description/meshes/Waist.STL"/>
+        iyy="0.292430846914939" iyz="-1.32037216353675E-18" izz="0.292430846914939" />
+    </inertial>
+    <visual>
+      <origin xyz="0 0 0" rpy="0 0 0" />
+      <geometry>
+        <mesh filename="file://$(find bpwr)/description/meshes/Waist.STL" />
       </geometry>
       <material name="blue">
-        <color rgba="0 0.819607843137255 0.933333333333333 1"/>
-      </material>
-    </visual>
-    <collision>
-      <origin xyz="0 0 0" rpy="0 0 0"/>
-      <geometry>
-        <mesh filename="file://$(find bpwr)/description/meshes/Waist.STL"/>
+        <color rgba="0 0.819607843137255 0.933333333333333 1" />
+      </material>
+    </visual>
+    <collision>
+      <origin xyz="0 0 0" rpy="0 0 0" />
+      <geometry>
+        <mesh filename="file://$(find bpwr)/description/meshes/Waist.STL" />
       </geometry>
     </collision>
@@ -30,22 +30,22 @@
   <link name="Hip_L">
     <inertial>
-      <origin xyz="1.14491749414469E-16 -0.145390450825359 -0.0291728991057009" rpy="0 0 0"/>
-      <mass value="0.607730964914872"/>
+      <origin xyz="1.14491749414469E-16 -0.145390450825359 -0.0291728991057009" rpy="0 0 0" />
+      <mass value="0.607730964914872" />
       <inertia ixx="0.0072795750548367" ixy="2.80537312130624E-18" ixz="-2.51690953028264E-19"
-               iyy="0.000340614101699668" iyz="-7.30812115544072E-05" izz="0.00756039905840226"/>
-    </inertial>
-    <visual>
-      <origin xyz="0 0 0" rpy="0 0 0"/>
-      <geometry>
-        <mesh filename="file://$(find bpwr)/description/meshes/Hip_L.STL"/>
-      </geometry>
-      <material name="">
-        <color rgba="0.792156862745098 0.819607843137255 0.933333333333333 1"/>
-      </material>
-    </visual>
-    <collision>
-      <origin xyz="0 0 0" rpy="0 0 0"/>
-      <geometry>
-        <mesh filename="file://$(find bpwr)/description/meshes/Hip_L.STL"/>
+        iyy="0.000340614101699668" iyz="-7.30812115544072E-05" izz="0.00756039905840226" />
+    </inertial>
+    <visual>
+      <origin xyz="0 0 0" rpy="0 0 0" />
+      <geometry>
+        <mesh filename="file://$(find bpwr)/description/meshes/Hip_L.STL" />
+      </geometry>
+      <material name="">
+        <color rgba="0.792156862745098 0.819607843137255 0.933333333333333 1" />
+      </material>
+    </visual>
+    <collision>
+      <origin xyz="0 0 0" rpy="0 0 0" />
+      <geometry>
+        <mesh filename="file://$(find bpwr)/description/meshes/Hip_L.STL" />
       </geometry>
     </collision>
@@ -53,22 +53,22 @@
   <link name="Shin_L">
     <inertial>
-      <origin xyz="1.66533453693773E-16 -0.145390450825359 0.0108271008942993" rpy="0 0 0"/>
-      <mass value="0.607730964914872"/>
+      <origin xyz="1.66533453693773E-16 -0.145390450825359 0.0108271008942993" rpy="0 0 0" />
+      <mass value="0.607730964914872" />
       <inertia ixx="0.0072795750548367" ixy="1.12079399580689E-17" ixz="2.23616698075135E-19"
-               iyy="0.000340614101699668" iyz="-7.30812115544049E-05" izz="0.00756039905840226"/>
-    </inertial>
-    <visual>
-      <origin xyz="0 0 0" rpy="0 0 0"/>
-      <geometry>
-        <mesh filename="file://$(find bpwr)/description/meshes/Shin_L.STL"/>
-      </geometry>
-      <material name="">
-        <color rgba="0.792156862745098 0.819607843137255 0.933333333333333 1"/>
-      </material>
-    </visual>
-    <collision>
-      <origin xyz="0 0 0" rpy="0 0 0"/>
-      <geometry>
-        <mesh filename="file://$(find bpwr)/description/meshes/Shin_L.STL"/>
+        iyy="0.000340614101699668" iyz="-7.30812115544049E-05" izz="0.00756039905840226" />
+    </inertial>
+    <visual>
+      <origin xyz="0 0 0" rpy="0 0 0" />
+      <geometry>
+        <mesh filename="file://$(find bpwr)/description/meshes/Shin_L.STL" />
+      </geometry>
+      <material name="">
+        <color rgba="0.792156862745098 0.819607843137255 0.933333333333333 1" />
+      </material>
+    </visual>
+    <collision>
+      <origin xyz="0 0 0" rpy="0 0 0" />
+      <geometry>
+        <mesh filename="file://$(find bpwr)/description/meshes/Shin_L.STL" />
       </geometry>
     </collision>
@@ -76,22 +76,22 @@
   <link name="Wheel_L">
     <inertial>
-      <origin xyz="5.55111512312578E-17 0 0.0333783783783784" rpy="0 0 0"/>
-      <mass value="0.46495571273129"/>
+      <origin xyz="5.55111512312578E-17 0 0.0333783783783784" rpy="0 0 0" />
+      <mass value="0.46495571273129" />
       <inertia ixx="0.00127876689292999" ixy="5.42101086242752E-20" ixz="8.80537574413171E-19"
-               iyy="0.00127876689292999" iyz="-2.79073771248327E-19" izz="0.00250573430050322"/>
-    </inertial>
-    <visual>
-      <origin xyz="0 0 0" rpy="0 0 0"/>
-      <geometry>
-        <mesh filename="file://$(find bpwr)/description/meshes/Wheel_L.STL"/>
-      </geometry>
-      <material name="">
-        <color rgba="0.792156862745098 0.819607843137255 0.933333333333333 1"/>
-      </material>
-    </visual>
-    <collision>
-      <origin xyz="0 0 0" rpy="0 0 0"/>
-      <geometry>
-        <mesh filename="file://$(find bpwr)/description/meshes/Wheel_L.STL"/>
+        iyy="0.00127876689292999" iyz="-2.79073771248327E-19" izz="0.00250573430050322" />
+    </inertial>
+    <visual>
+      <origin xyz="0 0 0" rpy="0 0 0" />
+      <geometry>
+        <mesh filename="file://$(find bpwr)/description/meshes/Wheel_L.STL" />
+      </geometry>
+      <material name="">
+        <color rgba="0.792156862745098 0.819607843137255 0.933333333333333 1" />
+      </material>
+    </visual>
+    <collision>
+      <origin xyz="0 0 0" rpy="0 0 0" />
+      <geometry>
+        <mesh filename="file://$(find bpwr)/description/meshes/Wheel_L.STL" />
       </geometry>
     </collision>
@@ -99,22 +99,22 @@
   <link name="Hip_R">
     <inertial>
-      <origin xyz="1.64798730217797E-17 -0.145390450825359 -0.0291728991057009" rpy="0 0 0"/>
-      <mass value="0.607730964914872"/>
+      <origin xyz="1.64798730217797E-17 -0.145390450825359 -0.0291728991057009" rpy="0 0 0" />
+      <mass value="0.607730964914872" />
       <inertia ixx="0.0072795750548367" ixy="5.01443504774546E-19" ixz="5.42101086242752E-20"
-               iyy="0.000340614101699668" iyz="-7.30812115544088E-05" izz="0.00756039905840226"/>
-    </inertial>
-    <visual>
-      <origin xyz="0 0 0" rpy="0 0 0"/>
-      <geometry>
-        <mesh filename="file://$(find bpwr)/description/meshes/Hip_R.STL"/>
-      </geometry>
-      <material name="">
-        <color rgba="0.792156862745098 0.819607843137255 0.933333333333333 1"/>
-      </material>
-    </visual>
-    <collision>
-      <origin xyz="0 0 0" rpy="0 0 0"/>
-      <geometry>
-        <mesh filename="file://$(find bpwr)/description/meshes/Hip_R.STL"/>
+        iyy="0.000340614101699668" iyz="-7.30812115544088E-05" izz="0.00756039905840226" />
+    </inertial>
+    <visual>
+      <origin xyz="0 0 0" rpy="0 0 0" />
+      <geometry>
+        <mesh filename="file://$(find bpwr)/description/meshes/Hip_R.STL" />
+      </geometry>
+      <material name="">
+        <color rgba="0.792156862745098 0.819607843137255 0.933333333333333 1" />
+      </material>
+    </visual>
+    <collision>
+      <origin xyz="0 0 0" rpy="0 0 0" />
+      <geometry>
+        <mesh filename="file://$(find bpwr)/description/meshes/Hip_R.STL" />
       </geometry>
     </collision>
@@ -122,22 +122,22 @@
   <link name="Shin_R">
     <inertial>
-      <origin xyz="2.77555756156289E-16 -0.145390450825358 0.0108271008942994" rpy="0 0 0"/>
-      <mass value="0.607730964914872"/>
+      <origin xyz="2.77555756156289E-16 -0.145390450825358 0.0108271008942994" rpy="0 0 0" />
+      <mass value="0.607730964914872" />
       <inertia ixx="0.0072795750548367" ixy="-1.31595038685428E-17" ixz="-1.8223425135342E-19"
-               iyy="0.000340614101699669" iyz="-7.30812115544176E-05" izz="0.00756039905840226"/>
-    </inertial>
-    <visual>
-      <origin xyz="0 0 0" rpy="0 0 0"/>
-      <geometry>
-        <mesh filename="file://$(find bpwr)/description/meshes/Shin_R.STL"/>
-      </geometry>
-      <material name="">
-        <color rgba="0.792156862745098 0.819607843137255 0.933333333333333 1"/>
-      </material>
-    </visual>
-    <collision>
-      <origin xyz="0 0 0" rpy="0 0 0"/>
-      <geometry>
-        <mesh filename="file://$(find bpwr)/description/meshes/Shin_R.STL"/>
+        iyy="0.000340614101699669" iyz="-7.30812115544176E-05" izz="0.00756039905840226" />
+    </inertial>
+    <visual>
+      <origin xyz="0 0 0" rpy="0 0 0" />
+      <geometry>
+        <mesh filename="file://$(find bpwr)/description/meshes/Shin_R.STL" />
+      </geometry>
+      <material name="">
+        <color rgba="0.792156862745098 0.819607843137255 0.933333333333333 1" />
+      </material>
+    </visual>
+    <collision>
+      <origin xyz="0 0 0" rpy="0 0 0" />
+      <geometry>
+        <mesh filename="file://$(find bpwr)/description/meshes/Shin_R.STL" />
       </geometry>
     </collision>
@@ -145,22 +145,22 @@
   <link name="Wheel_R">
     <inertial>
-      <origin xyz="-1.0547118733939E-15 -6.10622663543836E-16 0.0333783783783783" rpy="0 0 0"/>
-      <mass value="0.46495571273129"/>
+      <origin xyz="-1.0547118733939E-15 -6.10622663543836E-16 0.0333783783783783" rpy="0 0 0" />
+      <mass value="0.46495571273129" />
       <inertia ixx="0.00127876689292999" ixy="5.42101086242752E-20" ixz="-2.317331240564E-19"
-               iyy="0.00127876689292999" iyz="-1.34164060110775E-20" izz="0.00250573430050322"/>
-    </inertial>
-    <visual>
-      <origin xyz="0 0 0" rpy="0 0 0"/>
-      <geometry>
-        <mesh filename="file://$(find bpwr)/description/meshes/Wheel_R.STL"/>
-      </geometry>
-      <material name="">
-        <color rgba="0.792156862745098 0.819607843137255 0.933333333333333 1"/>
-      </material>
-    </visual>
-    <collision>
-      <origin xyz="0 0 0" rpy="0 0 0"/>
-      <geometry>
-        <mesh filename="file://$(find bpwr)/description/meshes/Wheel_R.STL"/>
+        iyy="0.00127876689292999" iyz="-1.34164060110775E-20" izz="0.00250573430050322" />
+    </inertial>
+    <visual>
+      <origin xyz="0 0 0" rpy="0 0 0" />
+      <geometry>
+        <mesh filename="file://$(find bpwr)/description/meshes/Wheel_R.STL" />
+      </geometry>
+      <material name="">
+        <color rgba="0.792156862745098 0.819607843137255 0.933333333333333 1" />
+      </material>
+    </visual>
+    <collision>
+      <origin xyz="0 0 0" rpy="0 0 0" />
+      <geometry>
+        <mesh filename="file://$(find bpwr)/description/meshes/Wheel_R.STL" />
       </geometry>
     </collision>
@@ -169,50 +169,101 @@
   <!--   JOINTS              -->
   <!-- ===================== -->
-      <!-- <joint name="base_link_joint" type="fixed">
-        <parent link="base_link"/>
-        <child link="Wheel_R"/>
-        <origin xyz="0 0.182941 0"/>
-    </joint> -->
   <joint name="L_Hip_Joint" type="revolute">
-    <origin xyz="0.23 0.018797 -0.0050706" rpy="1.5708 0.97309 -1.5708"/>
-    <parent link="Waist"/>
-    <child link="Hip_L"/>
-    <axis xyz="0 0 1"/>
-    <limit lower="-1.57" upper="1.57" effort="50" velocity="10"/>
+    <origin xyz="0.23 0.018797 -0.0050706" rpy="1.5708 0.97309 -1.5708" />
+    <parent link="Waist" />
+    <child link="Hip_L" />
+    <axis xyz="0 0 1" />
+    <limit lower="-1.57" upper="1.57" effort="50" velocity="10" />
   </joint>
   <joint name="L_Shin_Joint" type="revolute">
-    <origin xyz="0 -0.317 0" rpy="-3.1416 0 -1.6808"/>
-    <parent link="Hip_L"/>
-    <child link="Shin_L"/>
-    <axis xyz="0 0 1"/>
-    <limit lower="-1.57" upper="1.57" effort="50" velocity="10"/>
-  </joint>
-  <joint name="Wheel_L" type="continuous">
-    <origin xyz="0 -0.317 0" rpy="0 0 1.2761"/>
-    <parent link="Shin_L"/>
-    <child link="Wheel_L"/>
-    <axis xyz="0 0 1"/>
-    <limit lower="-1.57" upper="1.57" effort="50" velocity="10"/>
+    <origin xyz="0 -0.317 0" rpy="-3.1416 0 -1.6808" />
+    <parent link="Hip_L" />
+    <child link="Shin_L" />
+    <axis xyz="0 0 1" />
+    <limit lower="-1.57" upper="1.57" effort="50" velocity="10" />
+  </joint>
+  <joint name="Wheel_L_Joint" type="continuous">
+    <origin xyz="0 -0.317 0" rpy="0 0 1.2761" />
+    <parent link="Shin_L" />
+    <child link="Wheel_L" />
+    <axis xyz="0 0 1" />
+    <limit lower="-1.57" upper="1.57" effort="50" velocity="10" />
   </joint>
   <joint name="R_Hip_Joint" type="revolute">
-    <origin xyz="-0.23 0.018797 -0.0050706" rpy="1.5708 -0.97309 1.5708"/>
-    <parent link="Waist"/>
-    <child link="Hip_R"/>
-    <axis xyz="0 0 1"/>
-    <limit lower="-1.57" upper="1.57" effort="50" velocity="10"/>
+    <origin xyz="-0.23 0.018797 -0.0050706" rpy="1.5708 -0.97309 1.5708" />
+    <parent link="Waist" />
+    <child link="Hip_R" />
+    <axis xyz="0 0 1" />
+    <limit lower="-1.57" upper="1.57" effort="50" velocity="10" />
   </joint>
   <joint name="R_Shin_Joint" type="revolute">
-    <origin xyz="0 -0.317 0" rpy="3.1416 0 1.6808"/>
-    <parent link="Hip_R"/>
-    <child link="Shin_R"/>
-    <axis xyz="0 0 1"/>
-    <limit lower="-1.57" upper="1.57" effort="50" velocity="10"/>
-  </joint>
-  <joint name="Wheel_R" type="continuous">
-    <origin xyz="0 -0.317 0" rpy="0 0 1.6915"/>
-    <parent link="Shin_R"/>
-    <child link="Wheel_R"/>
-    <axis xyz="0 0 1"/>
-    <limit lower="0" upper="0" effort="0" velocity="0"/>
-  </joint>
+    <origin xyz="0 -0.317 0" rpy="3.1416 0 1.6808" />
+    <parent link="Hip_R" />
+    <child link="Shin_R" />
+    <axis xyz="0 0 1" />
+    <limit lower="-1.57" upper="1.57" effort="50" velocity="10" />
+  </joint>
+  <joint name="Wheel_R_Joint" type="continuous">
+    <origin xyz="0 -0.317 0" rpy="0 0 1.6915" />
+    <parent link="Shin_R" />
+    <child link="Wheel_R" />
+    <axis xyz="0 0 1" />
+    <limit lower="0" upper="0" effort="0" velocity="0" />
+  </joint>
+  <joint name="base_to_waist" type="fixed">
+    <parent link="base_link" />
+    <child link="Waist" />
+    <origin xyz="0 0 0.55" rpy="0 0 0" />
+  </joint>
+  <!-- ===================== -->
+  <!--   GAZEBO REFERENCES   -->
+  <!-- ===================== -->
+  <gazebo reference="base_link">
+    <material>Gazebo/Gray</material>
+  </gazebo>
+  <gazebo reference="L_Hip_Joint">
+    <provideFeedback>true</provideFeedback>
+    <damping>2.0</damping>
+  </gazebo>
+  <gazebo reference="R_Hip_Joint">
+    <provideFeedback>true</provideFeedback>
+    <damping>2.0</damping>
+  </gazebo>
+  <gazebo reference="L_Shin_Joint">
+    <provideFeedback>true</provideFeedback>
+    <damping>2.0</damping>
+  </gazebo>
+  <gazebo reference="R_Shin_Joint">
+    <provideFeedback>true</provideFeedback>
+    <damping>2.0</damping>
+  </gazebo>
+  <gazebo reference="Wheel_L">
+    <provideFeedback>true</provideFeedback>
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