Commit message: Added joint transforms to rviz. Wheels rotates now.

File: src/my_bot/description/gazebo_control.xacro (robot description, xacro)
@@ -22,4 +22,16 @@
             <command_topic>cmd_vel</command_topic>
         </plugin>
+        <plugin name="gazebo_ros_joint_state_publisher"
+            filename="libgazebo_ros_joint_state_publisher.so">
+            <alwaysOn>true</alwaysOn>
+            <updateRate>50</updateRate>
+            <joint_name>Wheel_L_Joint</joint_name>
+            <joint_name>Wheel_R_Joint</joint_name>
+            <joint_name>L_Hip_Joint</joint_name>
+            <joint_name>R_Hip_Joint</joint_name>
+            <joint_name>L_Shin_Joint</joint_name>
+            <joint_name>R_Shin_Joint</joint_name>
+            <!-- Add every movable joint -->
+        </plugin>
     </gazebo>
 </robot>

File: src/my_bot/description/robot_core.xacro (robot description, xacro)
@@ -8,5 +8,5 @@
     <inertial>
       <origin xyz="-1.18888240640652E-16 -0.00507058467782265 -0.0187972227348701" rpy="0 0 0" />
-      <mass value="14.4540071153471" />
+      <mass value="6.4540071153471" />
       <inertia ixx="0.0700688932175611" ixy="-3.86937762023137E-19" ixz="-1.76854570708965E-20"
         iyy="0.292430846914939" iyz="-1.32037216353675E-18" izz="0.292430846914939" />

Commit message: update

File: src/my_bot/description/gazebo_control.xacro (robot description, xacro)
@@ -2,25 +2,19 @@
 <robot xmlns:xacro="http://www.ros.org/wiki/xacro">
     <gazebo>
-        <plugin name="diff_drive" filename="libgazebo_ros_diff_drive.so">
-            <!-- Wheel Joint Names -->
+        <!--<plugin name="diff_drive" filename="libgazebo_ros_diff_drive.so">
             <left_joint>Wheel_L_Joint</left_joint>
             <right_joint>Wheel_R_Joint</right_joint>
-            <!-- Wheel Geometry -->
-            <wheel_separation>0.46</wheel_separation>     <!-- distance between wheel centers -->
-            <wheel_diameter>0.25</wheel_diameter>        <!-- wheel diameter -->
-            <!-- Limits -->
+            <wheel_separation>0.46</wheel_separation>
+            <wheel_diameter>0.25</wheel_diameter>
             <max_wheel_torque>20</max_wheel_torque>
             <max_wheel_acceleration>10.0</max_wheel_acceleration>
-            <!-- Odometry / TF Frames -->
             <odometry_frame>odom</odometry_frame>
             <robot_base_frame>base_link</robot_base_frame>
-            <!-- Publishing Options -->
             <publish_odom>true</publish_odom>
             <publish_odom_tf>true</publish_odom_tf>
             <publish_wheel_tf>true</publish_wheel_tf>
-            <!-- Command Topic (default: cmd_vel) -->
             <command_topic>cmd_vel</command_topic>
-        </plugin>
-        <plugin name="gazebo_ros_joint_state_publisher"
+        </plugin> -->
+        <!-- <plugin name="gazebo_ros_joint_state_publisher"
             filename="libgazebo_ros_joint_state_publisher.so">
             <alwaysOn>true</alwaysOn>
@@ -32,6 +26,34 @@
             <joint_name>L_Shin_Joint</joint_name>
             <joint_name>R_Shin_Joint</joint_name>
-            <!-- Add every movable joint -->
-        </plugin>
+        </plugin> -->
+        <gazebo>
+            <plugin name="gazebo_ros2_control" filename="libgazebo_ros2_control.so" />
+        </gazebo>
     </gazebo>
+    <!-- ====================== ROS2_CONTROL INTERFACE ====================== -->
+    <ros2_control name="GazeboSystem" type="system">
+        <hardware>
+            <plugin>gazebo_ros2_control/GazeboSystem</plugin>
+        </hardware>
+        <!-- Knee joints -->
+        <joint name="L_Hip_Joint">
+            <command_interface name="effort" />
+            <state_interface name="position" />
+            <state_interface name="velocity" />
+        </joint>
+        <joint name="R_Hip_Joint">
+            <command_interface name="effort" />
+            <state_interface name="position" />
+            <state_interface name="velocity" />
+        </joint>
+        <!-- Wheels (example) -->
+        <joint name="Wheel_L_Joint">
+            <command_interface name="velocity" />
+            <state_interface name="velocity" />
+        </joint>
+        <joint name="Wheel_R_Joint">
+            <command_interface name="velocity" />
+            <state_interface name="velocity" />
+        </joint>
+    </ros2_control>
 </robot>

File: src/my_bot/description/robot.urdf.xacro (robot description, xacro)
@@ -1,5 +1,8 @@
 <?xml version="1.0"?>
-<robot xmlns:xacro="http://www.ros.org/wiki/xacro"  name="Assem1">
-  <xacro:include filename="robot_core.xacro"/>
-  <xacro:include filename="gazebo_control.xacro"/>
+<robot xmlns:xacro="http://www.ros.org/wiki/xacro" name="Assem1">
+  <xacro:include filename="robot_core.xacro" />
+  <xacro:include filename="gazebo_control.xacro" />
+  <xacro:include filename="imu.xacro" />
+  <xacro:include filename="lidar.xacro" />
+  <xacro:include filename="camera.xacro" />
 </robot>

File: src/my_bot/description/robot_core.xacro (robot description, xacro)
@@ -176,4 +176,13 @@
     <limit lower="-1.57" upper="1.57" effort="50" velocity="10" />
   </joint>
+  <!-- <transmission name="L_Hip_Joint_trans">
+    <type>transmission_interface/SimpleTransmission</type>
+    <joint name="L_Hip_Joint">
+      <hardwareInterface>hardware_interface/EffortJointInterface</hardwareInterface>
+    </joint>
+    <actuator name="L_Hip_Joint_motor">
+      <hardwareInterface>hardware_interface/EffortJointInterface</hardwareInterface>
+    </actuator>
+  </transmission> -->
   <joint name="L_Shin_Joint" type="revolute">
     <origin xyz="0 -0.317 0" rpy="-3.1416 0 -1.6808" />
@@ -183,4 +192,13 @@
     <limit lower="-1.57" upper="1.57" effort="50" velocity="10" />
   </joint>
+  <!-- <transmission name="L_Shin_Joint_trans">
+    <type>transmission_interface/SimpleTransmission</type>
+    <joint name="R_Hip_Joint">
+      <hardwareInterface>hardware_interface/EffortJointInterface</hardwareInterface>
+    </joint>
+    <actuator name="L_Shin_Joint_motor">
+      <hardwareInterface>hardware_interface/EffortJointInterface</hardwareInterface>
+    </actuator>
+  </transmission> -->
   <joint name="Wheel_L_Joint" type="continuous">
     <origin xyz="0 -0.317 0" rpy="0 0 1.2761" />
@@ -197,4 +215,13 @@
     <limit lower="-1.57" upper="1.57" effort="50" velocity="10" />
   </joint>
+  <!-- <transmission name="R_Hip_Joint_trans">
+    <type>transmission_interface/SimpleTransmission</type>
+    <joint name="R_Hip_Joint">
+      <hardwareInterface>hardware_interface/EffortJointInterface</hardwareInterface>
+    </joint>
+    <actuator name="R_Hip_Joint_motor">
+      <hardwareInterface>hardware_interface/EffortJointInterface</hardwareInterface>
+    </actuator>
+  </transmission> -->
   <joint name="R_Shin_Joint" type="revolute">
     <origin xyz="0 -0.317 0" rpy="3.1416 0 1.6808" />
@@ -204,4 +231,13 @@
     <limit lower="-1.57" upper="1.57" effort="50" velocity="10" />
   </joint>
+    <!-- <transmission name="R_Shin_Joint_trans">
+    <type>transmission_interface/SimpleTransmission</type>
+    <joint name="L_Hip_Joint">
+      <hardwareInterface>hardware_interface/EffortJointInterface</hardwareInterface>
+    </joint>
+    <actuator name="R_Shin_Joint_motor">
+      <hardwareInterface>hardware_interface/EffortJointInterface</hardwareInterface>
+    </actuator>
+  </transmission> -->
   <joint name="Wheel_R_Joint" type="continuous">
     <origin xyz="0 -0.317 0" rpy="0 0 1.6915" />
@@ -243,5 +279,5 @@
     <mu1>1.5</mu1>
     <mu2>1.0</mu2>
-     <material>Gazebo/Black</material>
+    <material>Gazebo/Black</material>
   </gazebo>
   <gazebo reference="Wheel_R">
